File: Kicad/HF PA Radio Interface/HF PA Radio Interface.kicad_sch (KiCad schematic)
At the start: 187 parts, among them J1 Conn_01x06, J10 Conn_01x03, J11 Conn_01x04, J12 Conn_01x02, J13 Conn_01x02, J14 Conn_01x02, J15 Conn_01x03, J16 Conn_01x04, J17 Conn_01x04, J18 Conn_01x04, J2 Conn_Coaxial, J3 Conn_Coaxial, J4 Conn_Coaxial, J5 Conn_01x05, J6 Conn_01x05, J7 Conn_01x04, J8 Conn_01x04, J9 Conn_01x04, K1 G2RL-1-E, Q1 BC848W, Q2 2N7002, Q3 DMG2305UX, U1 74LVC1G17, U10 74AHCT125, U2 74LVC74, U3 TLV9364, U4 ADS1015IDGS, U5 TLV9361, U6 MCP4728, U7 AP2204K-ADJ, U8 LTC1044, U9 74LVC1G17

Commit message: Updates to HF PA Interface and PA Power_V1
Parts:
- C19, C23, C30, C33, C35, C36, C37, C39: value 10n -> 100n
- C28, C32, C34: value 10uF -> 10u
- D1, D13, D14, D15, D24, D28, D3, D6, D7: value SMF4L5.0A -> PESD5Z5.0F
- D12: value SMF4L12.0A -> PESD5Z12
- D18: value ESD131-B1-W0201 -> SBD52C05L01
- D20, D22, D25, D26, D27, D4, D9: value SMF4L12A -> PESD5Z12
Connections:
- net +5V: now also Q3.3 (D); no longer Q3.2 (S)
- net at A1.39 (VSYS): now also Q3.2 (S); no longer Q3.3 (D)
Other:
- note added: "DC Fan"
- note added: "PWM Fan 1"
- note added: "PWM Fan 2"
- note added: "PWM Fan 3"
- moved on the sheet: Q3, R42
